File: KiCAD/flip32.sch (KiCad schematic (older format))
At the start: 55 parts, among them CON1 USB-MICRO-B, IC1 MMA8452Q, IC2 MIC5205, P1 VBAT, P10 CONN_01X02, P2 ESC OUT, P3 BEEPER, P4 ESC PWR, P5 RECV CHANNELS, P6 EXP HEADER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

Commit message: Removed unused accelormeter (MMA8452Q)
Parts:
- removed C1, C3: 0.1uF, ~, symbol C
- removed C2: 4.7uF, ~, symbol C
- removed IC1: MMA8452Q, ~, symbol MMA8452Q
- removed R12: R, ~, symbol R
Connections:
- wire segments 279 -> 261
- no-connect marks 54 -> 48
Other:
- note removed: "Accelerometer"
