File: KiCAD/$flip32.sch (KiCad schematic (older format))
At the start: 51 parts, among them CON1 USB-MICRO-B, IC2 MIC5205, P1 VBAT, P10 BOOT, P2 ESC OUT, P3 BEEPER, P4 RECV CHANNELS, P5 UART 1, P6 I2C, P7 UNUSED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

Commit message: Finished pcb layout for MPU9150
Connections:
- net UU1: no longer names the net of P7.1 (P1)
Changed lines of the file:
@@
 Sheet 1 1
 Title "Flip32+"
-Date "16 jul 2015"
+Date "17 jul 2015"
 Rev "1"
 Comp ""
@@
 Wire Wire Line
 	6900 4500 7000 4500
-Text Label 11550 5300 2    60   ~ 0
-UU1
 Text Label 11550 5400 2    60   ~ 0
 UU2
